Commit message: refactor: Replace `curtis_motor` URDF and ROS2 control definitions with `system_traction` and update the launch configuration.

File: description/ros2_control/system_traction.ros2_control.xacro (robot description, xacro)
@@ -1,14 +1,13 @@
 <?xml version="1.0"?>
 <robot xmlns:xacro="http://www.ros.org/wiki/xacro">
-  <xacro:macro name="curtis_motor_ros2_control" params="update_rate">
-    <ros2_control name="curtis_motor" type="actuator">
+  <xacro:macro name="system_traction_ros2_control" params="update_rate">
+    <ros2_control name="system_traction" type="actuator">
         <hardware>
-            <plugin>caddy_ai2_ros2_control_hardware_curtis_motor_driver/CurtisMotorHardwareInterface</plugin>
-            <param name="can_interface">vcan_motor_drv</param>
+            <plugin>caddy_ai2_ros2_control_system_traction_driver/SystemTractionHardwareInterface</plugin>
+            <param name="can_interface">can_trac_drv</param>
             <param name="update_rate">${update_rate}</param>
         </hardware>
-        <joint name="curtis_motor_joint">
+        <joint name="system_traction_joint">
             <command_interface name="velocity"/>
-            <!-- CurtisMotorDriver -->
             <state_interface name="velocity"/> <!-- speed -->
             <state_interface name="motor_rpm"/> <!-- motor_rpm -->

File: description/urdf/system_traction.urdf.xacro (robot description, xacro)
@@ -1,7 +1,7 @@
 <?xml version="1.0"?>
-<robot xmlns:xacro="http://www.ros.org/wiki/xacro" name="curtis_motor">
+<robot xmlns:xacro="http://www.ros.org/wiki/xacro" name="system_traction">
   <xacro:arg name="prefix" default="" />
   <!-- Import RRBot ros2_control description -->
-  <xacro:include filename="$(find caddy_ai2_ros2_control_hardware_curtis_motor_driver)/ros2_control/curtis_motor.ros2_control.xacro" />
+  <xacro:include filename="$(find caddy_ai2_ros2_control_system_traction_driver)/description/ros2_control/system_traction.ros2_control.xacro" />
   <!-- Used for fixing robot -->
 <!-- Used for fixing robot -->
@@ -22,12 +22,12 @@
     </visual>
   </link>
-  <joint name="curtis_motor_joint" type="revolute">
+  <joint name="system_traction_joint" type="revolute">
     <parent link="base_link"/>
-    <child link="curtis_motor_link"/>
+    <child link="system_traction_link"/>
     <origin xyz="0 0 0.1" rpy="0 0 0"/>
     <axis xyz="0 1 0"/>
     <limit effort="1000" velocity="1000" lower="-3.14" upper="3.14"/>
   </joint>
-  <link name="curtis_motor_link">
+  <link name="system_traction_link">
     <visual>
       <geometry>
@@ -39,4 +39,4 @@
     </visual>
   </link>
-  <xacro:curtis_motor_ros2_control update_rate="$(arg update_rate)"/>
+  <xacro:system_traction_ros2_control update_rate="$(arg update_rate)"/>
 </robot>
